Commit message: remove world links

File: prbt_workcell_description/urdf/workcell.urdf (robot description, URDF)
Before this commit: robot ur5e_workcell, 8 links, 7 joints
Links:
- removed link world
Joints:
- removed joint robot_cell_base_joint

File: ur_workcell_description/urdf/workcell.urdf (robot description, URDF)
Before this commit: robot ur5e_workcell, 8 links, 7 joints
Links:
- removed link world
Joints:
- removed joint robot_cell_base_joint
